File: hardware/chlorophyll-sensor-v2/chlorophyll-sensor-v2/chlorophyll-sensor-v2.kicad_pcb (KiCad board)
At the start: 2 copper layers, 20 x 20 mm, 22 parts, among them J2 Conn_01x07_Male, U1 MIC5317, U2 MIC5317, U3 TSL257, U4 MCP3561

Commit message: softw update
Routing:
- net GND: track 26.5 -> 27.4 mm
Other:
- board text added: "Maciej Lewandowski"
Changed lines of the file:
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@@
     (property "Sheetname" "")
     (attr smd)
-    (fp_text reference "C14" (at 0 -1.43) (layer "F.SilkS")
-      (effects (font (size 1 1) (thickness 0.15)))
+    (fp_text reference "C14" (at -2.2 0.35 90) (layer "F.SilkS")
+      (effects (font (size 0.6 0.6) (thickness 0.1)))
     )
     (fp_text value "0.1uF" (at 0 1.43) (layer "F.Fab")
@@
     (property "Sheetname" "")
     (attr smd)
-    (fp_text reference "FB1" (at 0 -1.43 90) (layer "F.SilkS")
-      (effects (font (size 1 1) (thickness 0.15)))
+    (fp_text reference "FB1" (at 1.6125 -1 90) (layer "F.SilkS")
+      (effects (font (size 0.6 0.6) (thickness 0.1)))
     )
     (fp_text value "FerriteBead_Small" (at 0 1.43 90) (layer "F.Fab")
@@
     (property "Sheetname" "")
     (attr smd)
-    (fp_text reference "C8" (at 0 -1.43 90) (layer "F.SilkS")
-      (effects (font (size 1 1) (thickness 0.15)))
+    (fp_text reference "C8" (at 2.2 0.0125 90) (layer "F.SilkS")
+      (effects (font (size 0.6 0.6) (thickness 0.1)))
     )
     (fp_text value "10uF" (at 0 1.43 90) (layer "F.Fab")
@@
     (property "Sheetname" "")
     (attr smd)
-    (fp_text reference "C2" (at -1.1 -1.93) (layer "F.SilkS")
-      (effects (font (size 1 1) (thickness 0.15)))
+    (fp_text reference "C2" (at 2.5125 -0.15) (layer "F.SilkS")
+      (effects (font (size 0.6 0.6) (thickness 0.1)))
     )
     (fp_text value "10uF" (at 0 1.43) (layer "F.Fab")
@@
     (property "Sheetname" "")
     (attr smd)
-    (fp_text reference "U1" (at 0.1 -1.2 unlocked) (layer "F.SilkS")
-      (effects (font (size 1 1) (thickness 0.15)))
+    (fp_text reference "U1" (at -1.5 -3.5 unlocked) (layer "F.SilkS")
+      (effects (font (size 0.6 0.6) (thickness 0.1)))
     )
     (fp_text value "MIC5317" (at 0 1 unlocked) (layer "F.Fab")
@@
     (property "Sheetname" "")
     (attr smd)
-    (fp_text reference "C7" (at 0 -1.43 90) (layer "F.SilkS")
-      (effects (font (size 1 1) (thickness 0.15)))
+    (fp_text reference "C7" (at 2.1125 -0.1 180) (layer "F.SilkS")
+      (effects (font (size 0.6 0.6) (thickness 0.1)))
     )
     (fp_text value "10uF" (at 0 1.43 90) (layer "F.Fab")
@@
     (property "Sheetname" "")
     (attr smd)
-    (fp_text reference "C4" (at 0 -1.43) (layer "F.SilkS")
-      (effects (font (size 1 1) (thickness 0.15)))
+    (fp_text reference "C4" (at 2.5 0.05) (layer "F.SilkS")
+      (effects (font (size 0.6 0.6) (thickness 0.1)))
     )
     (fp_text value "0.1uF" (at 0 1.43) (layer "F.Fab")
@@
     (property "Sheetname" "")
     (attr smd)
-    (fp_text reference "C3" (at 0 -1.43) (layer "F.SilkS")
-      (effects (font (size 1 1) (thickness 0.15)))
+    (fp_text reference "C3" (at -1.8125 1) (layer "F.SilkS")
+      (effects (font (size 0.6 0.6) (thickness 0.15)))
     )
     (fp_text value "0.1uF" (at 0 1.43) (layer "F.Fab")
@@
     (property "Sheetname" "")
     (attr smd)
-    (fp_text reference "R1" (at 0 -1.43 90) (layer "F.SilkS")
-      (effects (font (size 1 1) (thickness 0.15)))
+    (fp_text reference "R1" (at -2.25 0.2 90) (layer "F.SilkS")
+      (effects (font (size 0.6 0.6) (thickness 0.1)))
     )
     (fp_text value "0" (at 0.025 -0.3325 90) (layer "F.Fab")
@@
     (property "Sheetname" "")
     (attr smd)
-    (fp_text reference "C10" (at 2.5125 1.1 90) (layer "F.SilkS")
-      (effects (font (size 1 1) (thickness 0.15)))
+    (fp_text reference "C10" (at 2.6375 -0.60625 90) (layer "F.SilkS")
+      (effects (font (size 0.6 0.6) (thickness 0.1)))
     )
     (fp_text value "0.1uF" (at 0 1.43 90) (layer "F.Fab")
@@
     (property "Sheetname" "")
     (attr smd)
-    (fp_text reference "C5" (at 0 -1.43 90) (layer "F.SilkS")
-      (effects (font (size 1 1) (thickness 0.15)))
+    (fp_text reference "C5" (at 2.1125 0.15 180) (layer "F.SilkS")
+      (effects (font (size 0.6 0.6) (thickness 0.1)))
     )
     (fp_text value "0.1uF" (at 0 1.43 90) (layer "F.Fab")
@@
     (property "Sheetname" "")
     (attr exclude_from_pos_files)
-    (fp_text reference "JP1" (at 0 -1.8 90) (layer "F.SilkS")
-      (effects (font (size 1 1) (thickness 0.15)))
+    (fp_text reference "JP1" (at 0.875 1.75625 90) (layer "F.SilkS")
+      (effects (font (size 0.6 0.6) (thickness 0.1)))
     )
     (fp_text value "Jumper_3_Open" (at 0 1.9 90) (layer "F.Fab")
@@
       (effects (font (size 1 1) (thickness 0.15)))
     )
-    (fp_text user "1" (at -2.6 0 90) (layer "F.SilkS")
+    (fp_text user "1" (at 0.125 -1.74375 90) (layer "F.SilkS")
       (effects (font (size 1 1) (thickness 0.15)))
     )
@@
     (property "Sheetname" "")
     (attr smd)
-    (fp_text reference "C12" (at 0 -1.43) (layer "F.SilkS")
-      (effects (font (size 1 1) (thickness 0.15)))
+    (fp_text reference "C12" (at -2.1 -0.15 90) (layer "F.SilkS")
+      (effects (font (size 0.6 0.6) (thickness 0.1)))
     )
     (fp_text value "0.1uF" (at 0 1.43) (layer "F.Fab")
@@
     (property "Sheetname" "")
     (attr smd)
-    (fp_text reference "C1" (at 0 -1.43) (layer "F.SilkS")
-      (effects (font (size 1 1) (thickness 0.15)))
+    (fp_text reference "C1" (at -2.55 0.2) (layer "F.SilkS")
+      (effects (font (size 0.6 0.6) (thickness 0.1)))
     )
     (fp_text value "10uF" (at 0 1.43) (layer "F.Fab")
@@
     (property "Sheetname" "")
     (attr smd)
-    (fp_text reference "C9" (at 2.5625 0 90) (layer "F.SilkS")
-      (effects (font (size 1 1) (thickness 0.15)))
+    (fp_text reference "C9" (at 2.375 -0.10625 90) (layer "F.SilkS")
+      (effects (font (size 0.6 0.6) (thickness 0.1)))
     )
     (fp_text value "10uF" (at 0 1.43 90) (layer "F.Fab")
@@
     (property "Sheetname" "")
     (attr smd)
-    (fp_text reference "U4" (at 0 -6.85 unlocked) (layer "F.SilkS")
+    (fp_text reference "U4" (at -0.2 -0.25 unlocked) (layer "F.SilkS")
       (effects (font (size 1 1) (thickness 0.15)))
     )
@@
     (property "Sheetname" "")
     (attr smd)
-    (fp_text reference "U2" (at 0.1 -1.2 unlocked) (layer "F.SilkS")
-      (effects (font (size 1 1) (thickness 0.15)))
+    (fp_text reference "U2" (at -1.1875 -1.4 unlocked) (layer "F.SilkS")
+      (effects (font (size 0.6 0.6) (thickness 0.1)))
     )
     (fp_text value "MIC5317" (at 0 1 unlocked) (layer "F.Fab")
@@
     (property "Sheetname" "")
     (attr smd)
-    (fp_text reference "C11" (at 0 -1.43) (layer "F.SilkS")
-      (effects (font (size 1 1) (thickness 0.15)))
+    (fp_text reference "C11" (at -1.8625 0.1 90) (layer "F.SilkS")
+      (effects (font (size 0.6 0.6) (thickness 0.1)))
     )
     (fp_text value "0.1uF" (at 0 1.43) (layer "F.Fab")
@@
     (property "Sheetname" "")
     (attr smd)
-    (fp_text reference "C13" (at 0 -1.43) (layer "F.SilkS")
-      (effects (font (size 1 1) (thickness 0.15)))
+    (fp_text reference "C13" (at -2.2125 -0.2 90) (layer "F.SilkS")
+      (effects (font (size 0.6 0.6) (thickness 0.1)))
     )
     (fp_text value "0.1uF" (at 0 1.43) (layer "F.Fab")
@@
     (property "Sheetname" "")
     (attr smd)
-    (fp_text reference "C6" (at 0 -1.43 90) (layer "F.SilkS")
-      (effects (font (size 1 1) (thickness 0.15)))
+    (fp_text reference "C6" (at -2.3 0.0125 90) (layer "F.SilkS")
+      (effects (font (size 0.6 0.6) (thickness 0.1)))
     )
     (fp_text value "0.1uF" (at 0 1.43 90) (layer "F.Fab")
@@
     (property "Sheetname" "")
     (attr through_hole)
-    (fp_text reference "U3" (at 0 -5.8 90 unlocked) (layer "B.SilkS")
+    (fp_text reference "U3" (at -3.975 -0.14375 90 unlocked) (layer "B.SilkS")
       (effects (font (size 1 1) (thickness 0.15)) (justify mirror))
     )
@@
   )
   (gr_rect (start 106.7 101.8) (end 86.7 81.8) (layer "Edge.Cuts") (width 0.1) (fill none))
+  (gr_text "Maciej Lewandowski" (at 91.75 101) (layer "F.SilkS")
+    (effects (font (size 0.6 0.6) (thickness 0.1)))
+  )
   (dimension (type aligned) (layer "F.SilkS")
     (pts (xy 86.7 81.8) (xy 86.7 101.8))
@@
   (segment (start 96.9 87.95) (end 96.75 88.1) (width 0.4) (layer "F.Cu") (net 2))
   (segment (start 98.5875 83.5125) (end 98.575 83.5) (width 0.4) (layer "F.Cu") (net 2))
+  (segment (start 96.75 88.1) (end 96.75 83.75) (width 0.4) (layer "F.Cu") (net 2))
+  (segment (start 96.75 83.75) (end 97 83.5) (width 0.4) (layer "F.Cu") (net 2))
   (segment (start 100.65 87.95) (end 101.35 87.25) (width 0.4) (layer "F.Cu") (net 2))
   (segment (start 98.95 87.95) (end 98.95 91.5875) (width 0.4) (layer "F.Cu") (net 2))
@@
   (segment (start 101.35 87.25) (end 102.85 87.25) (width 0.4) (layer "F.Cu") (net 2))
   (segment (start 98.9375 93.0375) (end 98.925 93.05) (width 0.4) (layer "F.Cu") (net 2))
+  (segment (start 97 83.5) (end 98.575 83.5) (width 0.4) (layer "F.Cu") (net 2))
   (segment (start 98.9375 91.6) (end 98.9375 93.0375) (width 0.4) (layer "F.Cu") (net 2))
-  (segment (start 96.75 88.1) (end 96.75 85.325) (width 0.4) (layer "F.Cu") (net 2))
   (segment (start 100.65 94.85) (end 99.850895 94.85) (width 0.4) (layer "F.Cu") (net 2))
   (segment (start 98.45 87.95) (end 100.65 87.95) (width 0.4) (layer "F.Cu") (net 2))
-  (segment (start 96.75 85.325) (end 98.575 83.5) (width 0.4) (layer "F.Cu") (net 2))
   (segment (start 98.95 91.5875) (end 98.9375 91.6) (width 0.4) (layer "F.Cu") (net 2))
   (segment (start 98.45 87.95) (end 98.95 87.95) (width 0.4) (layer "F.Cu") (net 2))
