File: hardware/chlorophyll-sensor-v2/chlorophyll-sensor-v2/chlorophyll-sensor-v2.kicad_sch (KiCad schematic)
At the start: 23 parts, among them J1 Conn_01x01_Male, J2 Conn_01x07_Male, U1 MIC5317, U2 MIC5317, U3 TSL257, U4 MCP3561

Commit message: softw update
Other:
- moved on the sheet: U3
Changed lines of the file:
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@@
     (stroke (width 0) (type default) (color 0 0 0 0))
   )
-  (wire (pts (xy 101.6 77.47) (xy 111.76 77.47))
+  (wire (pts (xy 92.71 85.09) (xy 102.87 85.09))
     (stroke (width 0) (type default) (color 0 0 0 0))
   )
@@
     (stroke (width 0) (type default) (color 0 0 0 0))
   )
-  (wire (pts (xy 101.6 74.93) (xy 104.14 74.93))
+  (wire (pts (xy 92.71 82.55) (xy 95.25 82.55))
     (stroke (width 0) (type default) (color 0 0 0 0))
   )
@@
     (stroke (width 0) (type default) (color 0 0 0 0))
   )
-  (wire (pts (xy 101.6 80.01) (xy 111.76 80.01))
+  (wire (pts (xy 92.71 87.63) (xy 102.87 87.63))
     (stroke (width 0) (type default) (color 0 0 0 0))
   )
@@
     (effects (font (size 1.27 1.27)) (justify left bottom))
   )
-  (label "OUT" (at 104.14 74.93 0)
+  (label "OUT" (at 95.25 82.55 0)
     (effects (font (size 1.27 1.27)) (justify left bottom))
   )
@@
     (pin "9")
   )
-  (symbol (lib_id "power:VDDA") (at 111.76 77.47 0) (unit 1)
-    (in_bom yes) (on_board yes) (fields_autoplaced)
-    (property "Reference" "#PWR017" (id 0) (at 111.76 81.28 0)
-      (effects (font (size 1.27 1.27)) hide)
-    )
-    (property "Value" "VDDA" (id 1) (at 111.76 72.39 0))
-    (property "Footprint" "" (id 2) (at 111.76 77.47 0)
-      (effects (font (size 1.27 1.27)) hide)
-    )
-    (property "Datasheet" "" (id 3) (at 111.76 77.47 0)
+  (symbol (lib_id "power:VDDA") (at 102.87 85.09 0) (unit 1)
+    (in_bom yes) (on_board yes) (fields_autoplaced)
+    (property "Reference" "#PWR017" (id 0) (at 102.87 88.9 0)
+      (effects (font (size 1.27 1.27)) hide)
+    )
+    (property "Value" "VDDA" (id 1) (at 102.87 80.01 0))
+    (property "Footprint" "" (id 2) (at 102.87 85.09 0)
+      (effects (font (size 1.27 1.27)) hide)
+    )
+    (property "Datasheet" "" (id 3) (at 102.87 85.09 0)
       (effects (font (size 1.27 1.27)) hide)
     )
@@
     (pin "1")
   )
-  (symbol (lib_id "power:GNDA") (at 111.76 80.01 0) (unit 1)
-    (in_bom yes) (on_board yes) (fields_autoplaced)
-    (property "Reference" "#PWR018" (id 0) (at 111.76 86.36 0)
-      (effects (font (size 1.27 1.27)) hide)
-    )
-    (property "Value" "GNDA" (id 1) (at 111.76 85.09 0))
-    (property "Footprint" "" (id 2) (at 111.76 80.01 0)
-      (effects (font (size 1.27 1.27)) hide)
-    )
-    (property "Datasheet" "" (id 3) (at 111.76 80.01 0)
+  (symbol (lib_id "power:GNDA") (at 102.87 87.63 0) (unit 1)
+    (in_bom yes) (on_board yes) (fields_autoplaced)
+    (property "Reference" "#PWR018" (id 0) (at 102.87 93.98 0)
+      (effects (font (size 1.27 1.27)) hide)
+    )
+    (property "Value" "GNDA" (id 1) (at 102.87 92.71 0))
+    (property "Footprint" "" (id 2) (at 102.87 87.63 0)
+      (effects (font (size 1.27 1.27)) hide)
+    )
+    (property "Datasheet" "" (id 3) (at 102.87 87.63 0)
       (effects (font (size 1.27 1.27)) hide)
     )
@@
     (pin "1")
   )
-  (symbol (lib_id "components:TSL257") (at 96.52 78.74 0) (mirror x) (unit 1)
-    (in_bom yes) (on_board yes) (fields_autoplaced)
-    (property "Reference" "U3" (id 0) (at 92.71 76.1999 0)
+  (symbol (lib_id "components:TSL257") (at 87.63 86.36 0) (mirror x) (unit 1)
+    (in_bom yes) (on_board yes) (fields_autoplaced)
+    (property "Reference" "U3" (id 0) (at 83.82 83.8199 0)
       (effects (font (size 1.27 1.27)) (justify right))
     )
-    (property "Value" "TSL257" (id 1) (at 92.71 78.7399 0)
+    (property "Value" "TSL257" (id 1) (at 83.82 86.3599 0)
       (effects (font (size 1.27 1.27)) (justify right))
     )
-    (property "Footprint" "components:TSL257" (id 2) (at 96.52 78.74 0)
-      (effects (font (size 1.27 1.27)) hide)
-    )
-    (property "Datasheet" "" (id 3) (at 96.52 78.74 0)
-      (effects (font (size 1.27 1.27)) hide)
-    )
+    (property "Footprint" "components:TSL257" (id 2) (at 87.63 86.36 0)
+      (effects (font (size 1.27 1.27)) hide)
+    )
+    (property "Datasheet" "" (id 3) (at 87.63 86.36 0)
+      (effects (font (size 1.27 1.27)) hide)
+    )
