File: hardware/radiation_sensor/radiation_sensor/radiation_sensor.kicad_pcb (KiCad board)
At the start: 2 copper layers, 33 x 23 mm, 33 parts, among them IC1 LTC6242HVCGN#PBF, J1 Conn_01x04, U1 LM393

Commit message: softw update
Other:
- net class Default removed
